Commit message: update

File: ur_description/urdf/ur10_joint_limited_robot.urdf.xacro (robot description, xacro)
@@ -31,5 +31,5 @@
     <parent link="tool0"/>
     <child link="robotiq_arg2f_base_link"/>
-    <origin xyz="0.0 0.0 0.0" rpy="0.0 0.0 0.0"/>
+    <origin xyz="0.0 0.0 0.0" rpy="0.0 0.0 1.57"/>
   </joint>
 </robot>
