Commit message: update

File: ur_description/urdf/desk.xacro (robot description, xacro)
@@ -3,5 +3,5 @@
     <link name="desk_link">
       <visual name="iron_frame_visual">
-        <pose>1.8 0 0 1.5707 0 1.5707 </pose>
+        <pose>0.8 0 0 0 0 0 </pose>
         <material name="silver">
  			<color rgba="0.6 0.6 0.6 1"/>
@@ -12,5 +12,5 @@
       </visual>
       <collision name="iron_frame_collision">
-        <pose>1.8 0 0 1.5707 0 1.5707</pose>
+        <pose>0.8 0 0 0 0 0</pose>
         <geometry>
 		<mesh filename="package://ur_description/meshes/ur10/collision/desk.stl"/>
@@ -30,7 +30,7 @@
     </link>
     <joint name="desk_to_world" type="fixed">
-    	<parent link="base"/>
+    	<parent link="world"/>
     	<child link="desk_link"/>
-    	<origin xyz="1.4 0.64 0" rpy="3.14 0 0"/>
+    	<origin xyz="-0.58 -0.6 0.7" rpy="-1.5707 0 1.5707"/>
     </joint>
   </robot>

File: ur_description/urdf/ur10.urdf.xacro (robot description, xacro)
@@ -287,11 +287,6 @@
       -->
       <origin xyz="0 0 0" rpy="0 0 ${-pi}"/>
-      <parent link="${prefix}base"/>
-      <child link="${prefix}base_link"/>
-<!--
-      <origin xyz="0 0 0" rpy="0 0 ${-pi}"/>
       <parent link="${prefix}base_link"/>
       <child link="${prefix}base"/>
--->
     </joint>
     <!-- Frame coincident with all-zeros TCP on UR controller -->

File: ur_description/urdf/ur10_joint_limited_robot.urdf.xacro (robot description, xacro)
@@ -10,12 +10,12 @@
   <xacro:include filename="$(find ur_description)/urdf/workcell.xacro" />
   <!-- desk -->
-  <!--<xacro:include filename="$(find ur_description)/urdf/desk.xacro" />-->
+  <xacro:include filename="$(find ur_description)/urdf/desk.xacro" />
   <!-- iron_frame -->
-  <xacro:include filename="$(find ur_description)/urdf/iron_frame.xacro" />
+  <!--xacro:include filename="$(find ur_description)/urdf/iron_frame.xacro" /-->
   <!-- gripper -->
   <xacro:include filename="$(find robotiq_arg2f_model_visualization)/urdf/robotiq_arg2f_140_model.xacro" />
   <!-- arm -->
   <xacro:ur10_robot prefix="" joint_limited="true"
-		 shoulder_pan_lower_limit="${-pi}" shoulder_pan_upper_limit="${pi}"
+		 shoulder_pan_lower_limit="${-pi/3}" shoulder_pan_upper_limit="${pi}"
 		 shoulder_lift_lower_limit="${-pi}" shoulder_lift_upper_limit="${pi}"
 		 elbow_joint_lower_limit="${-pi}" elbow_joint_upper_limit="${pi}"
@@ -24,4 +24,10 @@
 		 wrist_3_lower_limit="${-pi}" wrist_3_upper_limit="${pi}"
 />
+  <link name="world" />
+  <joint name="world_joint" type="fixed">
+    <parent link="world" />
+    <child link = "base_link" />
+    <origin xyz="0.0 0.0 0.5" rpy="0.0 0.0 0.0" />
+  </joint>
   <joint name="gripper_joint" type="fixed">
     <parent link="tool0"/>

File: ur_description/urdf/workcell.xacro (robot description, xacro)
@@ -10,7 +10,7 @@
   </link>
   <joint name="world_to_floor" type="fixed">
-    <parent link="base_link" />
+    <parent link="world" />
     <child link="floor" />
-    <origin xyz="0.0 0.0 -0.5" rpy="0.0 0.0 0.0" />
+    <origin xyz="0.0 0.0 0.0" rpy="0.0 0.0 0.0" />
   </joint>
  </robot>
