Commit message: update commits

File: ur_description/urdf/ur10.urdf.xacro (robot description, xacro)
@@ -263,8 +263,9 @@
       </xacro:cylinder_inertial>
     </link>
+    <!-- ee_link add 20cm -->
     <joint name="${prefix}ee_fixed_joint" type="fixed">
       <parent link="${prefix}wrist_3_link" />
       <child link = "${prefix}ee_link" />
-      <origin xyz="0.0 ${wrist_3_length} 0.0" rpy="0.0 0.0 ${pi/2.0}" />
+      <origin xyz="0.0 ${wrist_3_length+0.20} 0.0" rpy="0.0 0.0 ${pi/2.0}" />
     </joint>
     <link name="${prefix}ee_link">

File: ur_description/urdf/ur10_joint_limited_robot.urdf.xacro (robot description, xacro)
@@ -26,10 +26,10 @@
     <parent link="world" />
     <child link = "base_link" />
-    <origin xyz="0.0 0.0 0.5" rpy="0.0 0.0 0.0" />
+    <origin xyz="0.0 0.0 0.0" rpy="0.0 0.0 0.0" />
   </joint>
   <joint name="gripper_joint" type="fixed">
     <parent link="tool0"/>
     <child link="robotiq_arg2f_base_link"/>
-    <origin xyz="0.0 0.0 0.0" rpy="0.0 0.0 1.57"/>
+    <origin xyz="0.0 0.0 0.0" rpy="0.0 0.0 ${pi/2}"/>
   </joint>
 </robot>

File: ur_description/urdf/ur10_robot.urdf.xacro (robot description, xacro)
@@ -14,5 +14,5 @@
     <parent link="world" />
     <child link = "base_link" />
-    <origin xyz="0.0 0.0 0.5" rpy="0.0 0.0 0.0" />
+    <origin xyz="0.0 0.0 0.0" rpy="0.0 0.0 0.0" />
   </joint>
 </robot>

Commit message: update

File: ur_description/urdf/ur10.urdf.xacro (robot description, xacro)
@@ -267,5 +267,5 @@
       <parent link="${prefix}wrist_3_link" />
       <child link = "${prefix}ee_link" />
-      <origin xyz="0.0 ${wrist_3_length+0.20} 0.0" rpy="0.0 0.0 ${pi/2.0}" />
+      <origin xyz="0.0 ${wrist_3_length} 0.0" rpy="0.0 0.0 ${pi/2.0}" />
     </joint>
     <link name="${prefix}ee_link">
@@ -287,6 +287,11 @@
       -->
       <origin xyz="0 0 0" rpy="0 0 ${-pi}"/>
+      <parent link="${prefix}base"/>
+      <child link="${prefix}base_link"/>
+<!--
+      <origin xyz="0 0 0" rpy="0 0 ${-pi}"/>
       <parent link="${prefix}base_link"/>
       <child link="${prefix}base"/>
+-->
     </joint>
     <!-- Frame coincident with all-zeros TCP on UR controller -->

File: ur_description/urdf/ur10_joint_limited_robot.urdf.xacro (robot description, xacro)
@@ -15,5 +15,5 @@
   <!-- arm -->
   <xacro:ur10_robot prefix="" joint_limited="true"
-		 shoulder_pan_lower_limit="${-pi}" shoulder_pan_upper_limit="${pi}"
+		 shoulder_pan_lower_limit="${-pi/6}" shoulder_pan_upper_limit="${pi}"
 		 shoulder_lift_lower_limit="${-pi}" shoulder_lift_upper_limit="${pi}"
 		 elbow_joint_lower_limit="${-pi}" elbow_joint_upper_limit="${pi}"
@@ -22,10 +22,4 @@
 		 wrist_3_lower_limit="${-pi}" wrist_3_upper_limit="${pi}"
 />
-  <link name="world" />
-  <joint name="world_joint" type="fixed">
-    <parent link="world" />
-    <child link = "base_link" />
-    <origin xyz="0.0 0.0 0.0" rpy="0.0 0.0 0.0" />
-  </joint>
   <joint name="gripper_joint" type="fixed">
     <parent link="tool0"/>

File: ur_description/urdf/workcell.xacro (robot description, xacro)
@@ -10,7 +10,7 @@
   </link>
   <joint name="world_to_floor" type="fixed">
-    <parent link="world" />
+    <parent link="base_link" />
     <child link="floor" />
-    <origin xyz="0.0 0.0 0.0" rpy="0.0 0.0 0.0" />
+    <origin xyz="0.0 0.0 -0.5" rpy="0.0 0.0 0.0" />
   </joint>
  </robot>

Commit message: update

File: ur_description/urdf/ur10.urdf.xacro (robot description, xacro)
@@ -267,5 +267,5 @@
       <parent link="${prefix}wrist_3_link" />
       <child link = "${prefix}ee_link" />
-      <origin xyz="0.0 ${wrist_3_length} 0.0" rpy="0.0 0.0 ${pi/2.0}" />
+      <origin xyz="0.0 ${wrist_3_length + 0.3} 0.0" rpy="0.0 0.0 ${pi/2.0}" />
     </joint>
     <link name="${prefix}ee_link">

Commit message: update

File: ur_description/urdf/ur10.urdf.xacro (robot description, xacro)
@@ -263,9 +263,9 @@
       </xacro:cylinder_inertial>
     </link>
-    <!-- ee_link add 20cm -->
+    <!-- ee_link add 30cm -->
     <joint name="${prefix}ee_fixed_joint" type="fixed">
       <parent link="${prefix}wrist_3_link" />
       <child link = "${prefix}ee_link" />
-      <origin xyz="0.0 ${wrist_3_length + 0.3} 0.0" rpy="0.0 0.0 ${pi/2.0}" />
+      <origin xyz="0.0 ${wrist_3_length + 0.30} 0.0" rpy="0.0 0.0 ${pi/2.0}" />
     </joint>
     <link name="${prefix}ee_link">
