Commit message: change description

File: car_with_ur10_description/urdf/ur10_joint_limited_robot.urdf.xacro (robot description, xacro)
@@ -8,5 +8,5 @@
   <xacro:include filename="$(find ur_description)/urdf/ur10.urdf.xacro" />
   <!-- workcell -->
-  <xacro:include filename="$(find ur_description)/urdf/workcell.xacro" />
+  <!--<xacro:include filename="$(find ur_description)/urdf/workcell.xacro" />-->
   <!-- desk -->
   <xacro:include filename="$(find ur_description)/urdf/desk.xacro" />
@@ -25,9 +25,4 @@
 />
   <link name="world" />
-  <joint name="world_joint" type="fixed">
-    <parent link="world" />
-    <child link = "base_link" />
-    <origin xyz="0.0 0.0 0.5" rpy="0.0 0.0 0.0" />
-  </joint>
   <joint name="gripper_joint" type="fixed">
     <parent link="tool0"/>
